Commit message: Imported upstream version '2.4.0' of 'upstream'

File: omni_base_description/robots/omni_base.urdf.xacro (robot description, xacro)
@@ -1,5 +1,5 @@
 <?xml version="1.0"?>
 <!--
-  Copyright (c) 2023 PAL Robotics S.L. All rights reserved.
+  Copyright (c) 2024 PAL Robotics S.L. All rights reserved.
   Licensed under the Apache License, Version 2.0 (the "License");
   you may not use this file except in compliance with the License.
@@ -11,34 +11,58 @@
   See the License for the specific language governing permissions and
   limitations under the License.
- -->
+-->
 <robot  xmlns:xacro="http://ros.org/wiki/xacro" name="omni_base" >
-  <xacro:arg name="use_sim" default="false"/>
-  <xacro:arg name="front_laser_model" default="sick-571"/> <!-- false, hokuyo, sick-551, sick-561, sick-571-->
-  <xacro:arg name="rear_laser_model" default="sick-571"/> <!-- false, hokuyo, sick-551, sick-561, sick-571-->
-  <xacro:arg name="multiple" default="false"/>
-  <xacro:arg name="public_sim" default="false"/>
+  <!-- ARGUMENTS -->
+  <!-- no-laser, hokuyo, sick-551, sick-561, sick-571-->
+  <xacro:arg name="front_laser_model" default="sick-571"/>
+  <!-- no-laser, hokuyo, sick-551, sick-561, sick-571-->
+  <xacro:arg name="rear_laser_model" default="sick-571"/>
+  <!-- false, true-->
+  <xacro:arg name="add_on_module" default="no-add-on"/>
+  <!-- Execution env config -->
+  <xacro:arg name="use_sim_time" default="false"/>
+  <xacro:arg name="is_multiple" default="false"/>
   <xacro:arg name="namespace" default=""/>
+  <xacro:arg name="is_public_sim" default="false"/>
+  <!-- PROPERTIES -->
+  <!-- HW configuration -->
   <xacro:property name="front_laser_model" value="$(arg front_laser_model)" />
   <xacro:property name="rear_laser_model" value="$(arg rear_laser_model)" />
-  <xacro:property name="is_multiple" value="$(arg multiple)" />
-  <xacro:property name="is_public_sim" value="$(arg public_sim)" />
-  <xacro:property name="nsp" value="$(arg namespace)" />
-  <xacro:if value="${front_laser_model not in ['false', 'sick-551', 'sick-561', 'sick-571', 'hokuyo']}">
+  <xacro:property name="add_on_module" value="$(arg add_on_module)"/>
+  <!-- HW configuration check -->
+  <xacro:if value="${front_laser_model not in ['no-laser', 'sick-551', 'sick-561', 'sick-571', 'hokuyo']}">
     <xacro:wrong_laser_model/>
   </xacro:if>
-  <xacro:if value="${rear_laser_model not in ['false', 'sick-551', 'sick-561', 'sick-571', 'hokuyo']}">
+  <xacro:if value="${rear_laser_model not in ['no-laser', 'sick-551', 'sick-561', 'sick-571', 'hokuyo']}">
     <xacro:wrong_laser_model/>
   </xacro:if>
-  <!-- The following included files set up definitions of parts of the robot body -->
+  <xacro:if value="${add_on_module not in ['no-add-on', 'rgbd-sensors']}">
+    <xacro:wrong_add_on_module/>
+  </xacro:if>
+  <!-- Execution env configuration -->
+  <xacro:property name="use_sim_time" default="$(arg use_sim_time)"/>
+  <xacro:property name="is_multiple" value="$(arg is_multiple)" />
+  <xacro:property name="namespace" value="$(arg namespace)" />
+  <xacro:property name="is_public_sim" value="$(arg is_public_sim)" />
+  <!-- INCLUDES -->
   <!-- Base -->
   <xacro:include filename="$(find omni_base_description)/urdf/base/base_sensors.urdf.xacro" />
-  <!-- Generic simulator_gazebo plugins -->
-  <xacro:include filename="$(find omni_base_description)/gazebo/gazebo.urdf.xacro" />
-  <!-- ros2_control -->
+  <!-- RGBD Sensors -->
+  <xacro:if value="${add_on_module == 'rgbd-sensors'}">
+    <xacro:include filename="$(find omni_base_description)/urdf/cameras_add_on/cameras_add_on.urdf.xacro" />
+  </xacro:if>
+  <!-- Materials for visualization -->
+  <xacro:include filename="$(find pal_urdf_utils)/urdf/materials.urdf.xacro" />
+  <!-- Utils for degree to radian conversion -->
+  <xacro:include filename="$(find pal_urdf_utils)/urdf/deg_to_rad.urdf.xacro" />
+  <!-- ROS 2 Control -->
   <xacro:include filename="$(find omni_base_description)/ros2_control/ros2_control.urdf.xacro" />
-  <xacro:omni_base_ros2_control use_sim="$(arg use_sim)" />
-  <!-- Materials for visualization -->
-  <xacro:include filename="$(find omni_base_description)/urdf/materials.urdf.xacro" />
+  <xacro:omni_base_ros2_control />
+  <!-- ROBOT DEFINITION -->
   <!-- Now we can start using the macros included above to define the actual robot -->
   <xacro:base_sensors name="base" front_laser_model="$(arg front_laser_model)" rear_laser_model="$(arg rear_laser_model)"/>
+  <!-- RGBD Sensors -->
+  <xacro:if value="${add_on_module == 'rgbd-sensors'}">
+    <xacro:cameras_add_on name="cameras_add_on" parent="base_link"/>
+  </xacro:if>
 </robot>

File: omni_base_description/ros2_control/ros2_control.urdf.xacro (robot description, xacro)
@@ -1,5 +1,5 @@
 <?xml version="1.0"?>
 <!--
-Copyright (c) 2023 PAL Robotics S.L. All rights reserved.
+Copyright (c) 2024 PAL Robotics S.L. All rights reserved.
 Licensed under the Apache License, Version 2.0 (the "License");
 you may not use this file except in compliance with the License.
@@ -12,17 +12,33 @@
 limitations under the License.
  -->
-<robot xmlns:xacro="http://ros.org/wiki/xacro"
-       name="omni_base" >
-<xacro:macro name="omni_base_ros2_control" params="use_sim:=^|false">
-    <xacro:include filename="$(find omni_base_description)/urdf/wheels/wheel.ros2_control.xacro"/>
-    <xacro:include filename="$(find omni_base_description)/urdf/sensors/sensors.ros2_control.xacro"/>
+<robot xmlns:xacro="http://ros.org/wiki/xacro" name="omni_base" >
+  <!-- INCLUDES -->
+  <xacro:include filename="$(find omni_base_description)/urdf/wheels/wheel.ros2_control.xacro"/>
+  <xacro:include filename="$(find omni_base_description)/urdf/sensors/sensors.ros2_control.xacro"/>
+  <!-- MACRO DEFINITION-->
+  <xacro:macro name="omni_base_ros2_control">
+    <!-- Init the ROS 2 control gazebo interface -->
+    <xacro:if value="${use_sim_time}">
+      <gazebo>
+        <plugin filename="libgazebo_ros2_control.so" name="gazebo_ros2_control">
+          <parameters>$(find omni_base_description)/ros2_control/gazebo_controller_manager_cfg.yaml</parameters>
+          <!-- <robot_sim_type>gazebo_ros2_control/GazeboSystem</robot_sim_type>
+          <control_period>0.001</control_period> -->
+        </plugin>
+      </gazebo>
+    </xacro:if>
+    <!-- ROS 2 control config-->
     <ros2_control name="ros2_control_omni_base_system" type="system">
-      <xacro:if value="$(arg use_sim)">
-        <xacro:ros2_control_imu name="base_imu_sensor"/>
+      <!-- Execution env config -->
+      <xacro:if value="${use_sim_time}">
+        <!-- HW interface; gazebo-->
         <hardware>
           <plugin>gazebo_ros2_control/GazeboSystem</plugin>
         </hardware>
+        <!-- IMU sensor (only in simulation)-->
+        <xacro:ros2_control_imu name="base_imu_sensor"/>
       </xacro:if>
-      <xacro:unless value="$(arg use_sim)">
+      <xacro:unless value="${use_sim_time}">
+        <!-- HW interface; robot control-->
         <hardware>
           <plugin>robot_control/RobotControl</plugin>

File: omni_base_description/urdf/base/base.urdf.xacro (robot description, xacro)
@@ -1,5 +1,5 @@
 <?xml version="1.0"?>
 <!--
-  Copyright (c) 2023 PAL Robotics S.L. All rights reserved.
+  Copyright (c) 2024 PAL Robotics S.L. All rights reserved.
   Licensed under the Apache License, Version 2.0 (the "License");
   you may not use this file except in compliance with the License.
@@ -11,10 +11,7 @@
   See the License for the specific language governing permissions and
   limitations under the License.
- -->
+-->
 <robot xmlns:xacro="http://ros.org/wiki/xacro">
-  <xacro:include filename="$(find omni_base_description)/urdf/deg_to_rad.xacro"/>
-  <xacro:include filename="$(find omni_base_description)/urdf/wheels/wheel.urdf.xacro"/>
-  <xacro:include filename="$(find omni_base_description)/urdf/base/antenna.urdf.xacro"/>
-  <xacro:include filename="$(find omni_base_description)/urdf/sensors/imu.urdf.xacro"/>
+  <!-- PROPERTIES -->
   <!-- Wheel characteristics -->
   <xacro:property name="wheel_radius"     value="0.0762"/>
@@ -25,6 +22,12 @@
   <xacro:property name="wheel_velocity"   value="1.0"/>
   <xacro:property name="suspension_sagital_separation" value="0.345"/>
+  <!-- INCLUDES -->
+  <xacro:include filename="$(find omni_base_description)/urdf/base/base.gazebo.xacro"/>
+  <xacro:include filename="$(find omni_base_description)/urdf/wheels/wheel.urdf.xacro"/>
+  <xacro:include filename="$(find omni_base_description)/urdf/objects/antenna.urdf.xacro"/>
+  <xacro:include filename="$(find omni_base_description)/urdf/objects/antenna.urdf.xacro"/>
+  <!-- MACRO DEFINITION-->
   <xacro:macro name="base" params="name">
-    <!-- Base footprint -->
+    <!-- Base -->
     <link name="${name}_link">
       <inertial>
@@ -62,4 +65,5 @@
       </collision>
     </link>
+    <!-- Base footprint -->
     <link name="${name}_footprint"/>
     <joint name="${name}_footprint_joint" type="fixed">
@@ -68,19 +72,4 @@
       <parent link="${name}_footprint"/>
     </joint>
-  <!-- gazebo parameters are given here for base_link through base_footprint -->
-    <gazebo reference="${name}_footprint">
-      <kp>100000000.0</kp>
-      <kd>10.0</kd>
-      <mu1>0.1</mu1>
-      <mu2>0.1</mu2>
-      <fdir1>1 0 0</fdir1>
-      <maxVel>10.0</maxVel>
-      <minDepth>0.0005</minDepth>
-      <laserRetro>0</laserRetro>
-    </gazebo>
-    <!-- IMU -->
-    <xacro:imu_sensor name="${name}_imu" parent="${name}_link" update_rate="100.0">
-      <origin xyz="-0.287 0 0.092163" rpy="0 0 ${90.0 * deg_to_rad}" />
-    </xacro:imu_sensor>
     <!-- Docking link -->
     <link name="${name}_dock_link">
@@ -114,8 +103,8 @@
     </joint>
     <!-- Antennas -->
-    <xacro:antenna name="base_antenna_right" parent="base_link" reflect="1">
+    <xacro:antenna name="${name}_antenna_right" parent="${name}_link" reflect="1">
       <origin xyz="-0.2015 -0.13 0.2165" rpy="0 0 0" />
     </xacro:antenna>
-    <xacro:antenna name="base_antenna_left" parent="base_link" reflect="-1">
+    <xacro:antenna name="${name}_antenna_left" parent="${name}_link" reflect="-1">
       <origin xyz="-0.2015 0.13 0.2165" rpy="0 0 0" />
     </xacro:antenna>
@@ -124,4 +113,6 @@
     <xacro:wheel side="rear_right"  sagital_reflect="1.0" frontal_reflect="-1.0" radius="${wheel_radius}" width="${wheel_width}" torque="${wheel_torque}" velocity="${wheel_velocity}" frontal_separation="${wheel_pair_separation}" sagital_separation="${suspension_sagital_separation}" parent="${name}_link"/>
     <xacro:wheel side="rear_left"   sagital_reflect="-1.0" frontal_reflect="-1.0" radius="${wheel_radius}" width="${wheel_width}" torque="${wheel_torque}" velocity="${wheel_velocity}" frontal_separation="${wheel_pair_separation}" sagital_separation="${suspension_sagital_separation}" parent="${name}_link"/>
+    <!-- Gazebo config-->
+    <xacro:base_gazebo name="${name}"/>
   </xacro:macro>
 </robot>

File: omni_base_description/urdf/base/base_sensors.urdf.xacro (robot description, xacro)
@@ -13,14 +13,15 @@
  -->
 <robot xmlns:xacro="http://ros.org/wiki/xacro">
+  <!-- INCLUDES -->
   <xacro:include filename="$(find omni_base_description)/urdf/base/base.urdf.xacro"/>
+  <xacro:include filename="$(find omni_base_description)/urdf/sensors/imu.urdf.xacro"/>
   <xacro:include filename="$(find omni_base_description)/urdf/sensors/hokuyo_urg_04lx_ug01_laser.urdf.xacro"/>
   <xacro:include filename="$(find omni_base_description)/urdf/sensors/sick_tim551_laser.urdf.xacro"/>
   <xacro:include filename="$(find omni_base_description)/urdf/sensors/sick_tim561_laser.urdf.xacro"/>
   <xacro:include filename="$(find omni_base_description)/urdf/sensors/sick_tim571_laser.urdf.xacro"/>
-  <xacro:include filename="$(find omni_base_description)/urdf/deg_to_rad.xacro"/>
-  <!-- Laser model can be: false, hokuyo, sick-551, sick-561, sick-571-->
+  <!-- LASER MACRO DEFINITION -->
   <xacro:macro name="laser_sensor" params="name parent model ros_topic *origin update_rate:=10">
     <xacro:if value="${model == 'sick-551'}">
-      <!-- Rear Laser:  Theoretic FOV = 270 -->
+      <!-- Rear Laser = Theoretic FOV = 270 -->
       <xacro:sick_tim551_laser name="${name}" parent="${parent}" ros_topic="${ros_topic}" update_rate="${update_rate}" min_angle="${-135 * deg_to_rad}" max_angle="${135 * deg_to_rad}" >
         <xacro:insert_block name="origin" />
@@ -28,5 +29,5 @@
     </xacro:if>
     <xacro:if value="${model == 'sick-561'}">
-      <!-- Rear Laser:  Theoretic FOV = 270 -->
+      <!-- Rear Laser = Theoretic FOV = 270 -->
       <xacro:sick_tim561_laser name="${name}" parent="${parent}" ros_topic="${ros_topic}" update_rate="${update_rate}" min_angle="${-135 * deg_to_rad}" max_angle="${135 * deg_to_rad}" >
         <xacro:insert_block name="origin" />
@@ -34,5 +35,5 @@
     </xacro:if>
     <xacro:if value="${model == 'sick-571'}">
-      <!-- Rear Laser:  Theoretic FOV = 270 -->
+      <!-- Rear Laser = Theoretic FOV = 270 -->
       <xacro:sick_tim571_laser name="${name}" parent="${parent}" ros_topic="${ros_topic}" update_rate="${update_rate}" min_angle="${-135 * deg_to_rad}" max_angle="${135 * deg_to_rad}" >
         <xacro:insert_block name="origin" />
@@ -40,5 +41,5 @@
     </xacro:if>
     <xacro:if value="${model == 'hokuyo'}">
-      <!-- Rear Laser:  Theoretic FOV = 240 -->
+      <!-- Rear Laser = Theoretic FOV = 240 -->
       <xacro:hokuyo_urg_04lx_ug01_laser name="${name}" parent="${parent}" ros_topic="${ros_topic}" update_rate="${update_rate}" min_angle="${-120 * deg_to_rad}" max_angle="${120 * deg_to_rad}" >
         <xacro:insert_block name="origin" />
@@ -46,13 +47,14 @@
     </xacro:if>
   </xacro:macro>
-  <!-- front_laser_model can be: false, hokuyo, sick-551, sick-561, sick-571-->
-  <!-- rear_laser_model can be: false, hokuyo, sick-551, sick-561, sick-571-->
-  <xacro:macro name="base_sensors" params=" name front_laser_model:=sick-561 rear_laser_model:=sick-561 laser_height:=0.13244">
+  <!-- MACRO DEFINITION -->
+  <!-- front_laser_model can be =false, hokuyo, sick-551, sick-561, sick-571-->
+  <!-- rear_laser_model can be =false, hokuyo, sick-551, sick-561, sick-571-->
+  <xacro:macro name="base_sensors" params="name front_laser_model:=sick-561 rear_laser_model:=sick-561 laser_height:=0.13244">
     <!-- Rear Laser Sensor -->
-    <xacro:laser_sensor name="${name}_rear_laser" parent="${name}" model="${rear_laser_model}" ros_topic="scan_rear_raw">
+    <xacro:laser_sensor name="${name}_rear_laser" parent="${name}_link" model="${rear_laser_model}" ros_topic="scan_rear_raw">
       <origin xyz="-0.27512 0.18297 ${laser_height}" rpy="${-180 * deg_to_rad} 0 ${135 * deg_to_rad}" />
     </xacro:laser_sensor>
     <!-- Front Laser Sensor -->
-    <xacro:laser_sensor name="${name}_front_laser" parent="${name}" model="${front_laser_model}" ros_topic="scan_front_raw">
+    <xacro:laser_sensor name="${name}_front_laser" parent="${name}_link" model="${front_laser_model}" ros_topic="scan_front_raw">
       <origin xyz="0.27512 -0.18297 ${laser_height}" rpy="${-180 * deg_to_rad} 0 ${-45 * deg_to_rad}" />
     </xacro:laser_sensor>
@@ -70,4 +72,8 @@
         </inertial>
     </link>
+    <!-- IMU -->
+    <xacro:imu_sensor name="${name}_imu" parent="${name}_link" update_rate="100.0">
+      <origin xyz="-0.287 0 0.092163" rpy="0 0 ${90.0 * deg_to_rad}" />
+    </xacro:imu_sensor>
     <xacro:base name="${name}"/>
   </xacro:macro>

File: omni_base_description/urdf/objects/antenna.urdf.xacro (robot description, xacro)
@@ -13,4 +13,5 @@
 -->
 <robot xmlns:xacro="http://ros.org/wiki/xacro">
+  <!-- MACRO DEFINITION -->
   <xacro:macro name="antenna" params="name parent *origin reflect:=1">
     <link name="${name}_link">

File: omni_base_description/urdf/sensors/hokuyo_urg_04lx_ug01_laser.gazebo.xacro (robot description, xacro)
@@ -13,4 +13,5 @@
  -->
 <robot xmlns:xacro="http://ros.org/wiki/xacro">
+  <!-- MACRO DEFINITION -->
   <xacro:macro name="hokuyo_urg_04lx_ug01_laser_gazebo" params="name ros_topic update_rate min_angle max_angle">
     <gazebo reference="${name}_link">

File: omni_base_description/urdf/sensors/hokuyo_urg_04lx_ug01_laser.urdf.xacro (robot description, xacro)
@@ -13,5 +13,7 @@
  -->
 <robot xmlns:xacro="http://ros.org/wiki/xacro">
+  <!-- INCLUDES -->
   <xacro:include filename="$(find omni_base_description)/urdf/sensors/hokuyo_urg_04lx_ug01_laser.gazebo.xacro" />
+  <!-- MACRO DEFINITION -->
   <xacro:macro name="hokuyo_urg_04lx_ug01_laser" params="name parent *origin ros_topic update_rate min_angle max_angle">
     <link name="${name}_link" type="laser">
@@ -40,8 +42,8 @@
       <axis xyz="0 1 0"/>
       <xacro:insert_block name="origin"/>
-      <parent link="${parent}_link"/>
+      <parent link="${parent}"/>
       <child  link="${name}_link"/>
     </joint>
-    <!-- gazebo extensions -->
+    <!-- Gazebo config -->
     <xacro:hokuyo_urg_04lx_ug01_laser_gazebo name="${name}" ros_topic="${ros_topic}" update_rate="${update_rate}" min_angle="${min_angle}" max_angle="${max_angle}" />
   </xacro:macro>

File: omni_base_description/urdf/sensors/imu.urdf.xacro (robot description, xacro)
@@ -13,4 +13,7 @@
  -->
 <robot xmlns:xacro="http://ros.org/wiki/xacro">
+  <!-- INCLUDES -->
+  <xacro:include filename="$(find omni_base_description)/urdf/sensors/imu.gazebo.xacro" />
+  <!-- MACRO DEFINITION -->
   <xacro:macro name="imu_sensor" params="name parent *origin update_rate">
     <link name="${name}_link">
@@ -26,27 +29,6 @@
       <xacro:insert_block name="origin"/>
     </joint>
-    <gazebo reference="${name}_link">
-      <sensor name="${name}_sensor" type="imu">
-        <always_on>1</always_on>
-        <update_rate>100.0</update_rate>
-        <imu>
-          <noise>
-            <type>gaussian</type>
-            <rate>
-              <mean>0.0</mean>
-              <stddev>2e-4</stddev>
-              <bias_mean>0.0000075</bias_mean>
-              <bias_stddev>0.0000008</bias_stddev>
-            </rate>
-            <accel>
-              <mean>0.0</mean>
-              <stddev>1.7e-2</stddev>
-              <bias_mean>0.1</bias_mean>
-              <bias_stddev>0.001</bias_stddev>
-            </accel>
-          </noise>
-        </imu>
-      </sensor>
-    </gazebo>
+    <!-- Gazebo config-->
+    <xacro:imu_gazebo name="${name}" update_rate="${update_rate}" />
   </xacro:macro>
 </robot>

File: omni_base_description/urdf/sensors/sensors.ros2_control.xacro (robot description, xacro)
@@ -13,4 +13,5 @@
  -->
 <robot xmlns:xacro="http://ros.org/wiki/xacro">
+  <!-- MACRO DEFINITION -->
   <xacro:macro name="ros2_control_imu" params="name">
     <sensor name="${name}">

File: omni_base_description/urdf/sensors/sick_tim551_laser.gazebo.xacro (robot description, xacro)
@@ -13,4 +13,5 @@
  -->
 <robot xmlns:xacro="http://ros.org/wiki/xacro">
+  <!-- MACRO DEFINITION -->
   <xacro:macro name="sick_tim551_laser_gazebo" params="name ros_topic update_rate min_angle max_angle">
     <gazebo reference="${name}_link">
@@ -37,5 +38,5 @@
             <type>gaussian</type>
             <mean>0.0</mean>
-            <stddev>0.06</stddev>
+            <stddev>0.01</stddev>
           </noise>
         </ray>

File: omni_base_description/urdf/sensors/sick_tim551_laser.urdf.xacro (robot description, xacro)
@@ -13,5 +13,7 @@
  -->
 <robot xmlns:xacro="http://ros.org/wiki/xacro">
+  <!-- INCLUDES -->
   <xacro:include filename="$(find omni_base_description)/urdf/sensors/sick_tim551_laser.gazebo.xacro" />
+  <!-- MACRO DEFINITION -->
   <xacro:macro name="sick_tim551_laser" params="name parent *origin ros_topic update_rate min_angle max_angle">
      <link name="${name}_link" type="laser">
@@ -40,5 +42,5 @@
       <axis xyz="0 1 0"/>
       <xacro:insert_block name="origin"/>
-      <parent link="${parent}_link"/>
+      <parent link="${parent}"/>
       <child  link="${name}_link"/>
     </joint>

File: omni_base_description/urdf/sensors/sick_tim561_laser.gazebo.xacro (robot description, xacro)
@@ -13,4 +13,5 @@
  -->
 <robot xmlns:xacro="http://ros.org/wiki/xacro">
+  <!-- MACRO DEFINITION -->
   <xacro:macro name="sick_tim561_laser_gazebo" params="name ros_topic update_rate min_angle max_angle">
     <gazebo reference="${name}_link">
@@ -37,5 +38,5 @@
             <type>gaussian</type>
             <mean>0.0</mean>
-            <stddev>0.06</stddev>
+            <stddev>0.01</stddev>
           </noise>
         </ray>

File: omni_base_description/urdf/sensors/sick_tim561_laser.urdf.xacro (robot description, xacro)
@@ -13,5 +13,7 @@
  -->
 <robot xmlns:xacro="http://ros.org/wiki/xacro">
+  <!-- INCLUDES -->
   <xacro:include filename="$(find omni_base_description)/urdf/sensors/sick_tim561_laser.gazebo.xacro" />
+  <!-- MACRO DEFINITION -->
   <xacro:macro name="sick_tim561_laser" params="name parent *origin ros_topic update_rate min_angle max_angle">
      <link name="${name}_link" type="laser">
@@ -40,5 +42,5 @@
       <axis xyz="0 1 0"/>
       <xacro:insert_block name="origin"/>
-      <parent link="${parent}_link"/>
+      <parent link="${parent}"/>
       <child  link="${name}_link"/>
     </joint>

File: omni_base_description/urdf/sensors/sick_tim571_laser.gazebo.xacro (robot description, xacro)
@@ -13,4 +13,5 @@
  -->
 <robot xmlns:xacro="http://ros.org/wiki/xacro">
+  <!-- MACRO DEFINITION -->
   <xacro:macro name="sick_tim571_laser_gazebo" params="name ros_topic update_rate min_angle max_angle">
     <gazebo reference="${name}_link">
@@ -37,5 +38,5 @@
             <type>gaussian</type>
             <mean>0.0</mean>
-            <stddev>0.06</stddev>
+            <stddev>0.01</stddev>
           </noise>
         </ray>

File: omni_base_description/urdf/sensors/sick_tim571_laser.urdf.xacro (robot description, xacro)
@@ -13,5 +13,7 @@
  -->
 <robot xmlns:xacro="http://ros.org/wiki/xacro">
+  <!-- INCLUDES -->
   <xacro:include filename="$(find omni_base_description)/urdf/sensors/sick_tim571_laser.gazebo.xacro" />
+  <!-- MACRO DEFINITION -->
   <xacro:macro name="sick_tim571_laser" params="name parent *origin ros_topic update_rate min_angle max_angle">
      <link name="${name}_link" type="laser">
@@ -40,5 +42,5 @@
       <axis xyz="0 1 0"/>
       <xacro:insert_block name="origin"/>
-      <parent link="${parent}_link"/>
+      <parent link="${parent}"/>
       <child  link="${name}_link"/>
     </joint>

File: omni_base_description/urdf/wheels/wheel.gazebo.xacro (robot description, xacro)
@@ -12,4 +12,5 @@
  -->
 <robot xmlns:xacro="http://ros.org/wiki/xacro">
+  <!-- MACRO DEFINITION -->
   <xacro:macro name="wheel_gazebo" params="side">
     <!-- Contact model for the wheel surface -->

File: omni_base_description/urdf/wheels/wheel.ros2_control.xacro (robot description, xacro)
@@ -13,4 +13,5 @@
  -->
 <robot xmlns:xacro="http://ros.org/wiki/xacro">
+  <!-- MACRO DEFINITION -->
   <xacro:macro name="ros2_control_wheel" params="side">
     <joint name="wheel_${side}_joint">
